File: rice-eclipse-mk-1-1/main.brd (EAGLE design)
At the start: 110.2 x 91.2 mm, 136 parts, among them IC1 LMV321LICTRT, IC2 LMV321LICTRT, IC3 LMV321LICTRT, IC4 LMV321LICTRT, IC5 UA78M, IC6 LMV321LICTRT, IC7 LMV321LICTRT, IC8 LMV321LICTRT, IC9 LMV321LICTRT, U1 LM1084ISX-5.0/NOPB, U2 THS4531IDRD8-M, U3 THS4531IDRD8-M, U4 THS4531IDRD8-M, U5 THS4531IDRD8-M, U6 1101M2S3CQE2, X1 2540-5

Commit message: Routed and messed with text.
Parts:
- removed X1: 2540-5, con-3m:PAK100/2500-5-40
- removed X5, X6: (no value), con-phoenix-250-extra:1770908
- added LC_IN1, LC_IN2: (no value), con-phoenix-250-extra:1770908
- added RPI_GPIO: 2540-5, con-3m:PAK100/2500-5-40
- moved X4 5.86 mm to (79.8, 72.9)
- moved U$6 4.83 mm to (3.56, 37.8)
- moved U$5 4.58 mm to (3.56, 24.9)
- moved U$4 4.57 mm to (3.81, 12.2)
- moved U$7 3.81 mm to (5.08, 48.3)
- moved R22 3.31 mm to (105.4, 80.5)
- moved R13 3.30 mm to (105.7, 43.9)
- moved R18 3.30 mm to (105.7, 55.4)
- moved R10 2.84 mm to (106.7, 19.1)
- moved R11 1.55 mm to (94.2, 15.2)
- moved C17 1.52 mm to (32.8, 21.3)
- moved R14 1.52 mm to (94.7, 29.7)
- moved R9 1.52 mm to (98.0, 15.2)
- moved R5 0.25 mm to (6.35, 77.7)
- renumbered X2 to PT_123_IN, X3 to TC_PT4_IN
Connections:
- net +5V_RPI: now also RPI_GPIO.2; no longer X1.2
- net ADC1_CS: now also RPI_GPIO.22; no longer X1.22
- net ADC2_CS: now also RPI_GPIO.24; no longer X1.24
- net ADC3_CS: now also RPI_GPIO.26; no longer X1.26
- net CTRL_SOLENOID_1: now also RPI_GPIO.11; no longer X1.11
- net CTRL_SOLENOID_2: now also RPI_GPIO.13; no longer X1.13
- net CTRL_SOLENOID_3: now also RPI_GPIO.15; no longer X1.15
- net GND: now also RPI_GPIO.6; no longer X1.6
- net IGNITION_RELAY: now also RPI_GPIO.16; no longer X1.16
- net LC_1_OUT+: now also LC_IN1.P$3, LC_IN1.P$7; no longer X6.P$3, X6.P$7
- net LC_1_OUT-: now also LC_IN1.P$4, LC_IN1.P$8; no longer X6.P$4, X6.P$8
- net LC_2_OUT+: now also LC_IN1.P$1, LC_IN1.P$5; no longer X6.P$1, X6.P$5
- net LC_2_OUT-: now also LC_IN1.P$2, LC_IN1.P$6; no longer X6.P$2, X6.P$6
- net LC_3_OUT+: now also LC_IN2.P$3, LC_IN2.P$7; no longer X5.P$3, X5.P$7
- net LC_3_OUT-: now also LC_IN2.P$4, LC_IN2.P$8; no longer X5.P$4, X5.P$8
- net LC_4_OUT+: now also LC_IN2.P$1, LC_IN2.P$5; no longer X5.P$1, X5.P$5
- net LC_4_OUT-: now also LC_IN2.P$2, LC_IN2.P$6; no longer X5.P$2, X5.P$6
- net MISO: now also RPI_GPIO.21; no longer X1.21
- net MOSI: now also RPI_GPIO.19; no longer X1.19
- net RPI_GPIO_1: now also RPI_GPIO.1; no longer X1.1
- net RPI_GPIO_10: now also RPI_GPIO.10; no longer X1.10
- net RPI_GPIO_12: now also RPI_GPIO.12; no longer X1.12
- net RPI_GPIO_14: now also RPI_GPIO.14; no longer X1.14
- net RPI_GPIO_17: now also RPI_GPIO.17; no longer X1.17
- net RPI_GPIO_18: now also RPI_GPIO.18; no longer X1.18
- net RPI_GPIO_20: now also RPI_GPIO.20; no longer X1.20
- net RPI_GPIO_25: now also RPI_GPIO.25; no longer X1.25
- net RPI_GPIO_27: now also RPI_GPIO.27; no longer X1.27
- net RPI_GPIO_28: now also RPI_GPIO.28; no longer X1.28
- net RPI_GPIO_29: now also RPI_GPIO.29; no longer X1.29
- net RPI_GPIO_3: now also RPI_GPIO.3; no longer X1.3
- net RPI_GPIO_30: now also RPI_GPIO.30; no longer X1.30
- net RPI_GPIO_31: now also RPI_GPIO.31; no longer X1.31
- net RPI_GPIO_32: now also RPI_GPIO.32; no longer X1.32
- net RPI_GPIO_33: now also RPI_GPIO.33; no longer X1.33
- net RPI_GPIO_34: now also RPI_GPIO.34; no longer X1.34
- net RPI_GPIO_35: now also RPI_GPIO.35; no longer X1.35
- net RPI_GPIO_36: now also RPI_GPIO.36; no longer X1.36
- net RPI_GPIO_37: now also RPI_GPIO.37; no longer X1.37
- net RPI_GPIO_38: now also RPI_GPIO.38; no longer X1.38
- net RPI_GPIO_39: now also RPI_GPIO.39; no longer X1.39
- net RPI_GPIO_4: now also RPI_GPIO.4; no longer X1.4
- net RPI_GPIO_40: now also RPI_GPIO.40; no longer X1.40
- net RPI_GPIO_5: now also RPI_GPIO.5; no longer X1.5
- net RPI_GPIO_7: now also RPI_GPIO.7; no longer X1.7
- net RPI_GPIO_8: now also RPI_GPIO.8; no longer X1.8
- net RPI_GPIO_9: now also RPI_GPIO.9; no longer X1.9
- net SCLK: now also RPI_GPIO.23; no longer X1.23
Routing:
- net RELAY_NEGATIVE: track 44.7 -> 39.8 mm
- net SOLENOID_2_NEGATIVE: track 38.6 -> 34.3 mm
- net SOLENOID_3_NEGATIVE: track 59.6 -> 55.8 mm
- net +12V: track 124.7 -> 121.0 mm
- net +10V: track 40.0 -> 37.1 mm
- net SOLENOID_1_NEGATIVE: track 63.2 -> 61.0 mm
- net +5V: track 69.1 -> 67.4 mm
- net GND: track 17.6 -> 16.7 mm

Commit message: Routed and tried to gen board.
Fixed cap sizes too.
Parts:
- C14, C15, C18, C21, C24, C27, C8, C9: device rcl:C0603 -> rcl:C0402K
- R26: value 470 -> 530
- R27: value 130 -> 113
- moved R5 1.02 mm to (6.35, 78.7)
- moved R54 0.25 mm to (66.8, 19.1)
- moved R6 0.25 mm to (2.29, 74.9)
- moved R44 0.25 mm to (55.1, 16.0)
- moved R47 0.25 mm to (49.3, 33.8)
Routing:
- net GND: track 16.7 -> 276.6 mm, vias 0 -> 17
- net +3V3_PT: track 0.00 -> 161.6 mm
- net +3V3: track 0.00 -> 125.7 mm, vias 0 -> 1
- net +3V3_LC: track 0.00 -> 116.3 mm
- net MOSI: track 0.00 -> 102.6 mm
- net +12V: track 121.0 -> 218.4 mm, vias 0 -> 1
- net +3V3_ADC: track 0.00 -> 88.8 mm
- net MISO: track 0.00 -> 83.1 mm, vias 0 -> 4
- net SCLK: track 0.00 -> 83.1 mm, vias 0 -> 1
- net ADC1_A0: track 0.00 -> 71.4 mm, vias 0 -> 2
- net ADC2_A7: track 0.00 -> 66.3 mm, vias 0 -> 1
- net ADC1_A1: track 0.00 -> 66.2 mm, vias 0 -> 3
- net ADC2_A6: track 0.00 -> 64.3 mm, vias 0 -> 2
- net ADC2_A5: track 0.00 -> 62.7 mm, vias 0 -> 1
- net ADC2_A4: track 0.00 -> 60.8 mm, vias 0 -> 1
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Other:
- board text added: "C Shannon Rev 1.0"
- board text added: "Rice Eclipse"
- board text added: "eclipse.rice.edu"
