File: rice-eclipse-mk-1-1-side/rice-eclipse-mk-1-1-side/sideboard.brd (EAGLE design)
At the start: 92.4 x 113 mm, 65 parts, among them IC1 MCP6N11R, IC2 MCP6N11R, IC3 LMV321LICTRT, IC4 MCP6N11R, IC5 LMV321LICTRT, IC6 LMV321LICTRT, IC7 MCP6N11R, IC8 LMV321LICTRT

Commit message: Added and routed.
Routing:
- net GND: track 0.00 -> 357.7 mm
- net +3V3: track 0.00 -> 355.9 mm
- net LC4_OUT1: track 0.00 -> 56.9 mm
- net LC1_OUT: track 0.00 -> 46.2 mm
- net N$30: track 0.00 -> 35.6 mm
- net N$9: track 0.00 -> 34.6 mm
- net N$29: track 0.00 -> 34.4 mm
- net N$4: track 0.00 -> 34.3 mm
- net N$32: track 0.00 -> 33.8 mm
- net N$23: track 0.00 -> 33.8 mm
- net N$14: track 0.00 -> 33.8 mm
- net N$1: track 0.00 -> 31.5 mm
- net N$2: track 0.00 -> 30.6 mm
- net LC3_OUT: track 0.00 -> 27.1 mm
- net LC2_OUT: track 0.00 -> 22.9 mm
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
Commit message: Rerouted with more stuff.
Parts:
- removed RRN1, RRO1, RRO2, RRO3, RRO4, RRP1: (no value), rcl:0204/7
- removed X10, X3, X6, X8: (no value), con-phoenix-254:2POL254
- added RZ1: (no value), pot:S64W
- RRN2, RRN3, RRN4, RRP2, RRP3, RRP4: device rcl:0204/7 -> rcl:R0805
- moved X7 2.84 mm to (34.3, 73.7), turned to 270 degrees
- moved C5 2.84 mm to (31.8, 77.5), turned to 180 degrees
- moved RAA4 1.80 mm to (57.1, 48.3)
- moved RAA5 1.27 mm to (55.9, 61.0)
- moved RRN4 1.27 mm to (49.5, 85.1)
- moved RRP4 1.27 mm to (49.5, 96.5)
Connections:
- removed net N$10: RRN1.2, RRO1.2, RRP1.1, X3.1
- removed net N$16: IC2.5, RG2.1, RRO2.1, X6.2
- removed net N$25: IC4.5, RG3.1, RRO3.1, X8.2
- removed net N$34: IC7.5, RG4.1, RRO4.1, X10.2
- net +3V3: now also RZ1.E; no longer RRP1.2
- net GND: now also RZ1.A; no longer RRN1.1
- net N$19: now also IC2.5, RG2.1; no longer RRO2.2, X6.1
- net N$28: now also IC4.5, RG3.1; no longer RRO3.2, X8.1
- net N$37: now also IC7.5, RG4.1; no longer RRO4.2, X10.1
- net N$8: now also RZ1.S; no longer RRO1.1, X3.2
Routing:
- net +3V3: track 355.9 -> 589.6 mm
- net N$29: track 34.4 -> 58.8 mm
- net N$9: track 34.6 -> 13.4 mm
- net N$21: track 21.5 -> 41.6 mm
- net N$34: track 16.5 -> 0.00 mm
- net N$19: track 13.8 -> 29.8 mm
- net N$25: track 15.5 -> 0.00 mm
- net N$16: track 15.5 -> 0.00 mm
- net N$12: track 21.4 -> 36.8 mm
- net N$37: track 13.8 -> 28.6 mm
- net N$28: track 13.8 -> 28.6 mm
- net N$10: track 13.8 -> 0.00 mm
- net LC4_OUT1: track 56.9 -> 49.3 mm
- net N$22: track 10.8 -> 3.68 mm
- net N$2: track 30.6 -> 37.0 mm
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- added copper zone on layer 16, net GND
