File: rice-eclipse-mk-1-1-side/rice-eclipse-mk-1-1-side/sideboard.sch (EAGLE design)
At the start: 65 parts, among them IC1 MCP6N11R, IC2 MCP6N11R, IC3 LMV321LICTRT, IC4 MCP6N11R, IC5 LMV321LICTRT, IC6 LMV321LICTRT, IC7 MCP6N11R, IC8 LMV321LICTRT

Commit message: Rerouted with more stuff.
Parts:
- removed RRN1, RRO1, RRO2, RRO3, RRO4, RRP1: (no value), rcl:R-US_0204/7
- removed X10, X3, X6, X8: (no value), con-phoenix-254:MPT2
- added RZ1: (no value), pot:TRIM_US-S64W
- RRN2, RRN3, RRN4, RRP2, RRP3, RRP4: device rcl:R-US_0204/7 -> rcl:R-US_R0805
Connections:
- removed net N$10: RRN1.2, RRO1.2, RRP1.1, X3-1.1
- removed net N$16: IC2.REF, RG2.1, RRO2.1, X6-2.1
- removed net N$25: IC4.REF, RG3.1, RRO3.1, X8-2.1
- removed net N$34: IC7.REF, RG4.1, RRO4.1, X10-2.1
- net +3V3: now also RZ1.E; no longer RRP1.2
- net GND: now also RZ1.A; no longer RRN1.1
- net N$19: now also IC2.REF, RG2.1; no longer RRO2.2, X6-1.1
- net N$28: now also IC4.REF, RG3.1; no longer RRO3.2, X8-1.1
- net N$37: now also IC7.REF, RG4.1; no longer RRO4.2, X10-1.1
- net N$8: now also RZ1.S; no longer RRO1.1, X3-2.1
