File: rice-eclipse-mk1-1/main.brd (EAGLE design)
At the start: 110.2 x 91.2 mm, 136 parts, among them IC1 LMV321LICTRT, IC2 LMV321LICTRT, IC3 LMV321LICTRT, IC4 LMV321LICTRT, IC5 UA78M, IC6 LMV321LICTRT, IC7 LMV321LICTRT, IC8 LMV321LICTRT, IC9 LMV321LICTRT, U1 LM1084ISX-5.0/NOPB, U2 THS4531IDRD8-M, U3 THS4531IDRD8-M, U4 THS4531IDRD8-M, U5 THS4531IDRD8-M, U6 1101M2S3CQE2

Commit message: Fixed board files maybe.
Parts:
- removed IC5: UA78M, texas-extra:TO220S
- removed LED1, LED2, LED3, LED4: (no value), led:LED5MM
- removed REG1: AP2210N-3.3TRG1, diodes-extra:SOT23
- removed U$1, U$4, U$5, U$6, U$7: 1991095, con-phoenix-500-extra:1991095
- removed U1: LM1084ISX-5.0/NOPB, texas-extra:TS3B
- added +10V_LED, +12V_LED, +3.3V_LED, +5V_LED: (no value), led:LED5MM
- added 10V_REG: UA78M, texas-extra:TO220S
- added 3.3V_REG: AP2210N-3.3TRG1, diodes-extra:SOT23
- added 5V_REG: LM1084ISX-5.0/NOPB, texas-extra:TS3B
- added PWR_DEBUG: (no value), con-phoenix-254:5POL254
- added PWR_IN, PWR_OUT1, PWR_OUT2, SOL+RELAY, SOLENOIDS: 1991095, con-phoenix-500-extra:1991095
- added RPI_DEBUG: (no value), con-phoenix-254:7POL254
- C14, C15, C18, C21, C24, C27, C8, C9: value 10nF -> 0.1UF; device rcl:C0402K -> rcl:C0603
- moved RPI_GPIO 69.2 mm to (103.4, 104.4)
- moved R24 60.4 mm to (153.2, 93.5)
- moved U5 59.8 mm to (152.9, 86.9)
- moved U$8 59.6 mm to (54.4, 110.2)
- moved R5 59.4 mm to (54.1, 114.0)
- moved R13 59.0 mm to (164.6, 47.2)
- moved R18 59.0 mm to (164.6, 58.7)
- moved R22 59.0 mm to (164.3, 83.8)
- moved R6 58.6 mm to (49.3, 110.0)
- moved LC_IN1 58.3 mm to (157.7, 40.9)
- moved R12 58.3 mm to (155.4, 42.9)
- moved R15 58.3 mm to (152.4, 43.4)
- moved R16 58.3 mm to (152.4, 54.6)
- moved R19 58.3 mm to (150.9, 59.7)
- moved R20 58.3 mm to (151.6, 71.9)
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Connections:
- net +10V: now also 10V_REG.3, 5V_REG.3, PWR_DEBUG.2, PWR_OUT1.A1, PWR_OUT1.B1; no longer IC5.3, U$4.A2, U$4.B2, U1.3
- net +12V: now also +12V_LED.A, 10V_REG.1, PWR_DEBUG.1, PWR_OUT1.A2, PWR_OUT1.B2; no longer IC5.1, LED1.A, U$4.A1, U$4.B1
- net +12V_DEBUG: now also PWR_IN.A1, PWR_IN.B1; no longer U$1.A1, U$1.B1
- net +3V3: now also +3.3V_LED.A, 3.3V_REG.2, PWR_DEBUG.4, PWR_OUT2.A1, PWR_OUT2.B1; no longer LED3.A, REG1.2
- net +5V: now also +5V_LED.A, 3.3V_REG.3, 5V_REG.2, 5V_REG.4, PWR_DEBUG.3, PWR_OUT2.A2, PWR_OUT2.B2; no longer LED2.A, REG1.3, U$5.A1, U$5.B1, U1.2, U1.4
- net ADC1_CS: now also RPI_DEBUG.4
- net ADC2_CS: now also RPI_DEBUG.3
- net ADC3_CS: now also RPI_DEBUG.2
- net GND: now also +10V_LED.K, 10V_REG.2, 3.3V_REG.1, 5V_REG.1, PWR_DEBUG.5, PWR_IN.A2, PWR_IN.B2, RPI_DEBUG.1; no longer IC5.2, LED4.A, REG1.1, U$1.A2, U$1.B2, U$5.A2, U$5.B2, U1.1
- net MISO: now also RPI_DEBUG.6
- net MOSI: now also RPI_DEBUG.5
- net N$1: now also +12V_LED.K; no longer LED1.K
- net N$2: now also +5V_LED.K; no longer LED2.K
- net N$3: now also +3.3V_LED.K; no longer LED3.K
- net N$9: now also +10V_LED.A; no longer LED4.K
- net RELAY_NEGATIVE: now also SOL+RELAY.A1, SOL+RELAY.B1; no longer U$6.A1, U$6.B1
- net SCLK: now also RPI_DEBUG.7
- net SOLENOID_1_NEGATIVE: now also SOL+RELAY.A2, SOL+RELAY.B2; no longer U$6.A2, U$6.B2
- net SOLENOID_2_NEGATIVE: now also SOLENOIDS.A1, SOLENOIDS.B1; no longer U$7.A1, U$7.B1
- net SOLENOID_3_NEGATIVE: now also SOLENOIDS.A2, SOLENOIDS.B2; no longer U$7.A2, U$7.B2
Routing:
- net GND: track 276.6 -> 8.20 mm, vias 17 -> 0
- net +3V3_PT: track 161.6 -> 0.00 mm
- net +3V3_LC: track 116.3 -> 0.00 mm
- net MOSI: track 102.6 -> 0.00 mm
- net +3V3_ADC: track 88.8 -> 0.00 mm
- net MISO: track 83.1 -> 0.00 mm, vias 4 -> 0
- net SCLK: track 83.1 -> 0.00 mm, vias 1 -> 0
- net +3V3: track 125.7 -> 51.6 mm, vias 1 -> 0
- net ADC1_A0: track 71.4 -> 0.00 mm, vias 2 -> 0
- net ADC2_A7: track 66.3 -> 0.00 mm, vias 1 -> 0
- net ADC1_A1: track 66.2 -> 0.00 mm, vias 3 -> 0
- net +12V: track 218.4 -> 153.9 mm, vias 1 -> 0
- net ADC2_A6: track 64.3 -> 0.00 mm, vias 2 -> 0
- net ADC2_A5: track 62.7 -> 0.00 mm, vias 1 -> 0
- net ADC2_A4: track 60.8 -> 0.00 mm, vias 1 -> 0
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Other:
- board size 110.2 x 91.2 mm -> 170.1 x 119.4 mm

Commit message: Fixed major known bugs in board design.
* 5V power rail for AA voltage follower.
* 10V rail to power PT connector.
Connections:
- net +10V: now also PT_123_IN.P$10, PT_123_IN.P$12, PT_123_IN.P$2, PT_123_IN.P$4, PT_123_IN.P$6, PT_123_IN.P$8, TC_PT4_IN.P$12, TC_PT4_IN.P$6
- net +12V: no longer PT_123_IN.P$10, PT_123_IN.P$12, PT_123_IN.P$2, PT_123_IN.P$4, PT_123_IN.P$6, PT_123_IN.P$8, TC_PT4_IN.P$12, TC_PT4_IN.P$6
- net +3V3_PT: no longer C18.1, C21.1, C24.1, C27.1, IC6.5, IC7.5, IC8.5, IC9.5
- net +5V: now also C18.1, C21.1, C24.1, C27.1, IC6.5, IC7.5, IC8.5, IC9.5
Changed lines of the file:
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@@
 </signal>
 <signal name="+12V">
-<contactref element="PT_123_IN" pad="P$12"/>
-<contactref element="PT_123_IN" pad="P$6"/>
-<contactref element="PT_123_IN" pad="P$8"/>
-<contactref element="PT_123_IN" pad="P$2"/>
-<contactref element="PT_123_IN" pad="P$10"/>
-<contactref element="PT_123_IN" pad="P$4"/>
-<contactref element="TC_PT4_IN" pad="P$12"/>
-<contactref element="TC_PT4_IN" pad="P$6"/>
 <contactref element="10V_REG" pad="1"/>
 <contactref element="C17" pad="+"/>
@@
 <wire x1="25.908" y1="76.18194375" x2="4.7" y2="54.97394375" width="1.016" layer="1"/>
 <wire x1="4.7" y1="54.97394375" x2="4.7" y2="30.5446375" width="1.016" layer="1"/>
-<wire x1="121.11" y1="5.762" x2="121.11" y2="10.762" width="0" layer="19" extent="1-1"/>
-<wire x1="97.836" y1="10.508" x2="121.11" y2="10.762" width="0" layer="19" extent="1-1"/>
-<wire x1="97.836" y1="5.508" x2="97.836" y2="10.508" width="0" layer="19" extent="1-1"/>
-<wire x1="92.836" y1="10.508" x2="97.836" y2="10.508" width="0" layer="19" extent="1-1"/>
-<wire x1="87.836" y1="10.508" x2="92.836" y2="10.508" width="0" layer="19" extent="1-1"/>
-<wire x1="92.836" y1="5.508" x2="97.836" y2="5.508" width="0" layer="19" extent="1-1"/>
-<wire x1="87.836" y1="5.508" x2="87.836" y2="10.508" width="0" layer="19" extent="1-1"/>
-<wire x1="56.388" y1="22.86" x2="87.836" y2="10.508" width="0" layer="19" extent="1-1"/>
 <wire x1="32.004" y1="39.116" x2="56.388" y2="22.86" width="0" layer="19" extent="1-1"/>
 <wire x1="28.956" y1="8.128" x2="15.748" y2="26.416" width="0" layer="19" extent="1-1"/>
@@
 <wire x1="33.528" y1="73.322" x2="33.698" y2="73.152" width="1.016" layer="1"/>
 <wire x1="33.698" y1="73.152" x2="39.37" y2="73.152" width="1.016" layer="1"/>
+<contactref element="IC6" pad="5"/>
+<contactref element="C18" pad="1"/>
+<contactref element="IC7" pad="5"/>
+<contactref element="C21" pad="1"/>
+<contactref element="IC9" pad="5"/>
+<contactref element="C27" pad="1"/>
+<contactref element="IC8" pad="5"/>
+<contactref element="C24" pad="1"/>
+<wire x1="118.364" y1="54.698" x2="121.986" y2="55.148" width="0" layer="19" extent="1-1"/>
+<wire x1="106.238" y1="54.64" x2="118.364" y2="54.698" width="0" layer="19" extent="1-1"/>
+<wire x1="104.14" y1="54.698" x2="106.238" y2="54.64" width="0" layer="19" extent="1-1"/>
+<wire x1="90.744" y1="55.656" x2="104.14" y2="54.698" width="0" layer="19" extent="1-1"/>
+<wire x1="87.376" y1="55.206" x2="90.744" y2="55.656" width="0" layer="19" extent="1-1"/>
+<wire x1="70.932" y1="56.926" x2="87.376" y2="55.206" width="0" layer="19" extent="1-1"/>
+<wire x1="67.818" y1="56.476" x2="70.932" y2="56.926" width="0" layer="19" extent="1-1"/>
+<wire x1="56.896" y1="46.228" x2="67.818" y2="56.476" width="0" layer="19" extent="1-1"/>
 <wire x1="39.624" y1="57.658" x2="56.896" y2="46.228" width="0" layer="19" extent="1-1"/>
 <wire x1="30.3276" y1="56.134" x2="38.608" y2="56.134" width="0" layer="19" extent="1-1"/>
@@
 <wire x1="23.368" y1="55.372" x2="23.368" y2="52.832" width="1.016" layer="16"/>
 <wire x1="23.368" y1="52.832" x2="32.004" y2="44.196" width="1.016" layer="16"/>
+<contactref element="PT_123_IN" pad="P$8"/>
+<contactref element="PT_123_IN" pad="P$2"/>
+<contactref element="PT_123_IN" pad="P$10"/>
+<contactref element="PT_123_IN" pad="P$4"/>
+<contactref element="PT_123_IN" pad="P$12"/>
+<contactref element="PT_123_IN" pad="P$6"/>
+<contactref element="TC_PT4_IN" pad="P$12"/>
+<contactref element="TC_PT4_IN" pad="P$6"/>
+<wire x1="121.11" y1="5.762" x2="121.11" y2="10.762" width="0" layer="19" extent="1-1"/>
+<wire x1="97.836" y1="10.508" x2="121.11" y2="10.762" width="0" layer="19" extent="1-1"/>
+<wire x1="97.836" y1="5.508" x2="97.836" y2="10.508" width="0" layer="19" extent="1-1"/>
+<wire x1="92.836" y1="10.508" x2="97.836" y2="10.508" width="0" layer="19" extent="1-1"/>
+<wire x1="92.836" y1="5.508" x2="97.836" y2="5.508" width="0" layer="19" extent="1-1"/>
+<wire x1="87.836" y1="10.508" x2="92.836" y2="10.508" width="0" layer="19" extent="1-1"/>
+<wire x1="87.836" y1="5.508" x2="92.836" y2="5.508" width="0" layer="19" extent="1-1"/>
+<wire x1="47.918" y1="38.1" x2="87.836" y2="10.508" width="0" layer="19" extent="1-1"/>
 <wire x1="38.608" y1="44.196" x2="47.918" y2="38.1" width="0" layer="19" extent="1-1"/>
 <wire x1="31.496" y1="8.128" x2="15.312" y2="31.202" width="0" layer="19" extent="1-1"/>
@@
 <contactref element="JP2" pad="2"/>
 <contactref element="R38" pad="1"/>
-<contactref element="IC6" pad="5"/>
-<contactref element="C18" pad="1"/>
 <contactref element="IC2" pad="5"/>
 <contactref element="C9" pad="1"/>
 <contactref element="R44" pad="1"/>
-<contactref element="IC7" pad="5"/>
-<contactref element="C21" pad="1"/>
-<contactref element="IC8" pad="5"/>
-<contactref element="C24" pad="1"/>
-<contactref element="IC9" pad="5"/>
-<contactref element="C27" pad="1"/>
 <contactref element="IC3" pad="5"/>
 <contactref element="C14" pad="1"/>
@@
 <contactref element="C15" pad="1"/>
 <contactref element="R58" pad="1"/>
-<wire x1="118.364" y1="54.698" x2="121.986" y2="55.148" width="0" layer="19" extent="1-1"/>
-<wire x1="106.238" y1="54.64" x2="118.364" y2="54.698" width="0" layer="19" extent="1-1"/>
-<wire x1="104.14" y1="54.698" x2="106.238" y2="54.64" width="0" layer="19" extent="1-1"/>
-<wire x1="90.744" y1="55.656" x2="104.14" y2="54.698" width="0" layer="19" extent="1-1"/>
-<wire x1="87.376" y1="55.206" x2="90.744" y2="55.656" width="0" layer="19" extent="1-1"/>
-<wire x1="100.33" y1="38.608" x2="104.14" y2="54.698" width="0" layer="19" extent="1-1"/>
-<wire x1="104.902" y1="33.616" x2="100.33" y2="38.608" width="0" layer="19" extent="1-1"/>
-<wire x1="107.254" y1="34.066" x2="104.902" y2="33.616" width="0" layer="19" extent="1-1"/>
+<wire x1="121.92" y1="34.886" x2="124.018" y2="35.336" width="0" layer="19" extent="1-1"/>
+<wire x1="118.11" y1="36.576" x2="121.92" y2="34.886" width="0" layer="19" extent="1-1"/>
+<wire x1="107.254" y1="34.066" x2="118.11" y2="36.576" width="0" layer="19" extent="1-1"/>
+<wire x1="104.902" y1="33.616" x2="107.254" y2="34.066" width="0" layer="19" extent="1-1"/>
+<wire x1="100.33" y1="38.608" x2="104.902" y2="33.616" width="0" layer="19" extent="1-1"/>
 <wire x1="90.236" y1="34.32" x2="100.33" y2="38.608" width="0" layer="19" extent="1-1"/>
 <wire x1="87.884" y1="33.87" x2="90.236" y2="34.32" width="0" layer="19" extent="1-1"/>
 <wire x1="84.328" y1="36.576" x2="87.884" y2="33.87" width="0" layer="19" extent="1-1"/>
-<wire x1="118.11" y1="36.576" x2="107.254" y2="34.066" width="0" layer="19" extent="1-1"/>
-<wire x1="121.92" y1="34.886" x2="118.11" y2="36.576" width="0" layer="19" extent="1-1"/>
-<wire x1="124.018" y1="35.336" x2="121.92" y2="34.886" width="0" layer="19" extent="1-1"/>
 <wire x1="70.424" y1="33.558" x2="84.328" y2="36.576" width="0" layer="19" extent="1-1"/>
 <wire x1="67.818" y1="33.108" x2="70.424" y2="33.558" width="0" layer="19" extent="1-1"/>
 <wire x1="64.77" y1="36.576" x2="67.818" y2="33.108" width="0" layer="19" extent="1-1"/>
-<wire x1="70.932" y1="56.926" x2="87.376" y2="55.206" width="0" layer="19" extent="1-1"/>
-<wire x1="67.818" y1="56.476" x2="70.932" y2="56.926" width="0" layer="19" extent="1-1"/>
-<wire x1="61.214" y1="53.086" x2="67.818" y2="56.476" width="0" layer="19" extent="1-1"/>
+<wire x1="61.214" y1="53.086" x2="64.77" y2="36.576" width="0" layer="19" extent="1-1"/>
 </signal>
 <signal name="+3V3_LC">

Commit message: Added our library to Eagle. Updated the LC circuit.
Parts:
- removed C10, C11: 1UF, rcl:C0603
- removed JP3: (no value), pinhead:1X02
- removed LC_IN1, LC_IN2: (no value), con-phoenix-250-extra:1770908
- removed R10, R13, R18, R22: (no value), pot-extra:PTD902
- removed R11, R14, R15, R16, R19, R20, R23, R24: 20K, rcl:R0603
- removed R12, R17, R21, R9: 33K, rcl:R0603
- removed U2, U3, U4, U5: THS4531IDRD8-M, texas-extra:D8-M
- added C30, C32, C34: 1UF, rcl:C0805
- added C31, C33, C35: 6.8nF, rcl:C0805
- added CAL1: (no value), con-phoenix-254:2POL254
- added IC10, IC11, IC12, IC5: MCP6N11R, microchip-extra:SO-8
- added JP4: (no value), pinhead:1X02
- added RF1, RF2, RF3, RF4, RF5: 20K, rcl:0204/7
- added RG1, RG2, RG3, RG4: 200, rcl:0204/7
- added RZ1, RZ2, RZ3, RZ4: (no value), pot:S64W
- added U$1, U$4: 1991118, con-phoenix-500-extra:1991118
- C12: device rcl:C0603 -> rcl:C0805
- C13: value 1UF -> 6.8nF; device rcl:C0603 -> rcl:C0805
- moved C12 26.4 mm to (140.7, 92.5), turned to 180 degrees
- moved C13 7.38 mm to (149.1, 93.0), turned to 180 degrees
- moved X4 1.30 mm to (135.1, 86.4)
- moved C3 1.27 mm to (114.6, 83.3)
- moved ADC1 0.51 mm to (122.7, 86.4)
- moved R25 0.36 mm to (115.1, 92.2)
Connections:
- removed net N$14: R10.2-1, R11.1, U2.8
- removed net N$15: R12.1, U3.7
- removed net N$16: R13.2-1, R15.1, U3.8
- removed net N$17: R10.1-1, R14.1, U2.1
- removed net N$18: R13.1-1, R16.1, U3.1
- removed net N$19: R17.1, U4.7
- removed net N$23: R22.2-1, R23.1, U5.8
- new net CAL: IC10.8, IC11.8, IC12.8
- new net N$39: C33.1, IC11.1, RF3.2, RG3.2
- new net N$40: C31.2, IC5.6, RF1.1
- new net N$41: C31.1, IC5.1, RF1.2, RG1.2
- new net N$42: IC5.5, RG1.1, RZ1.S
- new net N$43: IC11.5, RG3.1, RZ3.S
- new net N$45: C35.2, IC12.6, RF4.1
- new net N$46: C35.1, IC12.1, RF4.2, RG4.2
- new net N$47: IC12.5, RG4.1, RZ4.S
- net +3V3: now also JP4.1; no longer JP3.1
- net +3V3_LC: now also C30.1, C32.1, C34.1, CAL1.1, IC10.7, IC11.7, IC12.7, IC5.7, JP4.2, RZ1.E, RZ2.E, RZ3.E, RZ4.E; no longer C10.1, C11.1, C13.1, JP3.2, R12.2, R17.2, R21.2, R9.2, U2.3, U3.3, U4.3, U5.3
- net ADC1_A0: no longer R11.2, U2.5
- net ADC1_A1: no longer R14.2, U2.4
- net ADC1_A2: no longer R15.2, U3.5
- net ADC1_A3: no longer R16.2, U3.4
- net ADC1_A4: no longer R19.2, U4.5
- net ADC1_A5: no longer R20.2, U4.4
- net ADC1_A6: no longer R23.2, U5.5
- net ADC1_A7: no longer R24.2, U5.4
- net GND: now also C30.2, C32.2, C34.2, IC10.4, IC11.4, IC12.4, IC5.4, RF5.2, RZ1.A, RZ2.A, RZ3.A, RZ4.A; no longer C10.2, C11.2, C13.2, U2.6, U3.6, U4.6, U5.6
- net LC_1_OUT+: now also IC5.3, U$4.A3, U$4.B3; no longer LC_IN1.P$3, LC_IN1.P$7, R10.2-2
- net LC_1_OUT-: now also IC5.2, U$4.A4, U$4.B4; no longer LC_IN1.P$4, LC_IN1.P$8, R10.1-2
- net LC_2_OUT+: now also IC10.3, U$4.A1, U$4.B1; no longer LC_IN1.P$1, LC_IN1.P$5, R13.2-2
- net LC_2_OUT-: now also IC10.2, U$4.A2, U$4.B2; no longer LC_IN1.P$2, LC_IN1.P$6, R13.1-2
- net LC_3_OUT+: now also IC11.3, U$1.A3, U$1.B3; no longer LC_IN2.P$3, LC_IN2.P$7, R18.2-2
- net LC_3_OUT-: now also IC11.2, U$1.A4, U$1.B4; no longer LC_IN2.P$4, LC_IN2.P$8, R18.1-2
- net LC_4_OUT+: now also IC12.3, U$1.A1, U$1.B1; no longer LC_IN2.P$1, LC_IN2.P$5, R22.2-2
- net LC_4_OUT-: now also IC12.2, U$1.A2, U$1.B2; no longer LC_IN2.P$2, LC_IN2.P$6, R22.1-2
- net N$13: now also CAL1.2, IC5.8, RF5.1; no longer R9.1, U2.7
- net N$20: now also C13.2, IC10.6, RF2.1; no longer R18.2-1, R19.1, U4.8
- net N$21: now also C13.1, IC10.1, RF2.2, RG2.2; no longer R18.1-1, R20.1, U4.1
- net N$22: now also IC10.5, RG2.1, RZ2.S; no longer R21.1, U5.7
- net N$24: now also C33.2, IC11.6, RF3.1; no longer R22.1-1, R24.1, U5.1
Other:
- board text added: "C Shannon Rev 1.1"
- board text removed: "C Shannon Rev 1.0"

Commit message: Minor improvements to board.
Parts:
- removed RF5: 20K, rcl:0204/7
- added D6: 1N4004, diode:DO41-10
- added R10: 500k, rcl:R0805
- added R9: 10k, rcl:R0805
- added RPD1: 20K, rcl:R0805
- added SOLENOIDS2: 1991095, con-phoenix-500-extra:1991095
- added U$5: IRF740, transistor-power:TO220BV
- C1, C14, C15, C18, C2, C21, C24, C27, C3, C8, C9: device rcl:C0603 -> rcl:C0805
- C19, C22, C25, C28: value (none) -> 470nF; device rcl:C025-025X050 -> rcl:C0805
- C20, C23, C26, C29: value (none) -> 4.7nF; device rcl:C025-025X050 -> rcl:C0805
- CAL1: device con-phoenix-254:2POL254 -> pinhead:1X02
- R1, R2, R25, R29, R3, R30, R4, R5, R6, R7, R8: device rcl:R0603 -> rcl:R0805
- R26, R27, R28, R35: device resistor:R0603 -> resistor:R0805
- R34, R36, R37, R38, R39, R42, R43, R44, R45, R46, R47, R48, R49, R50, R51, R52, R53, R54, R56, R57, R58, R59, RF1, RF2, RF3, RF4, RG1, RG2, RG3, RG4: device rcl:0204/7 -> rcl:R0805
- R40: value ? -> 150K; device rcl:0204/7 -> rcl:R0805
- R41: value ? -> 1.5K; device rcl:0204/7 -> rcl:R0805
- moved CAL1 86.4 mm to (190.8, 65.3), turned to 0 degrees
- moved D1 3.57 mm to (31.0, 99.8)
Connections:
- new net CTRL_SOLENOID_4: R9.1
- new net N$14: R10.1, R9.2, U$5.G
- new net N$15: SOLENOIDS2.A2, SOLENOIDS2.B2
- new net SOLENOID_4_NEGATIVE: D6.A, SOLENOIDS2.A1, SOLENOIDS2.B1, U$5.D
- net +12V: now also D6.C
- net GND: now also R10.2, RPD1.2, U$5.S; no longer RF5.2
- net N$13: now also RPD1.1; no longer RF5.1
Routing:
- net SOLENOID_4_NEGATIVE: track 0.00 -> 24.9 mm
- net N$15: track 0.00 -> 8.20 mm
- net GND: track 8.20 -> 0.00 mm
- net RELAY_NEGATIVE: track 29.4 -> 36.2 mm
- net SOLENOID_2_NEGATIVE: track 66.4 -> 71.9 mm
- net SOLENOID_3_NEGATIVE: track 83.3 -> 88.2 mm
- net SOLENOID_1_NEGATIVE: track 44.4 -> 49.0 mm

Commit message: Moved onto board. Preliminary power routing.
Parts:
- removed CAL1: (no value), pinhead:1X02
- removed PT_123_IN, TC_PT4_IN: (no value), con-phoenix-250-extra:1770924
- removed U$1, U$4: 1991118, con-phoenix-500-extra:1991118
- added LC1/2, LC3/4, PT1/2, PT3/4, THERMOCOUPLES: 1991118, con-phoenix-500-extra:1991118
- added LC_EN/CAL: (no value), pinhead:1X02
- C19, C22, C25, C28: value 470nF -> 68nF
- C20, C23, C26, C29: value 4.7nF -> 680pF
- R31, R32, R33, R55: value 10 -> 22; device rcl:R0603 -> rcl:R0805
- R34, R36, R38, R42, R44, R53, R56, R58: value ? -> 20K
- R37, R43, R47, R49, R51, R52, R57: value ? -> 150K
- R39, R45, R54, R59: value ? -> 3K
- R46, R48, R50: value ? -> 1.5K
- moved JP4 221.1 mm to (120.4, 94.2)
- moved RZ1 165.7 mm to (129.8, 15.2), turned to 90 degrees
- moved C31 145.4 mm to (139.4, 10.2), turned to 180 degrees
- moved IC5 141.9 mm to (139.4, 16.8), turned to 90 degrees
- moved C30 140.2 mm to (134.9, 23.1), turned to 0 degrees
- moved RF1 139.2 mm to (141.2, 22.9), turned to 0 degrees
- moved RG1 138.8 mm to (146.3, 21.1), turned to 270 degrees
- moved RPD1 106.6 mm to (147.6, 100.6)
- moved RZ4 104.1 mm to (145.8, 88.4), turned to 90 degrees
- moved RZ3 93.1 mm to (128.5, 51.8), turned to 90 degrees
- moved C34 86.2 mm to (152.4, 94.7)
- moved C32 81.8 mm to (135.6, 61.2)
- moved RF4 79.7 mm to (159.3, 94.5)
- moved C35 79.3 mm to (153.9, 81.5)
- moved RG2 76.0 mm to (149.1, 35.8), turned to 270 degrees
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Connections:
- removed net N$13: CAL1.2, IC5.8, RPD1.1
- removed net N$20: C13.2, IC10.6, RF2.1
- removed net N$24: C33.2, IC11.6, RF3.1
- removed net N$40: C31.2, IC5.6, RF1.1
- removed net N$45: C35.2, IC12.6, RF4.1
- removed net RPI_GPIO_18: RPI_GPIO.18
- net +10V: now also PT1/2.A1, PT1/2.A3, PT1/2.B1, PT1/2.B3, PT3/4.A1, PT3/4.A3, PT3/4.B1, PT3/4.B3; no longer PT_123_IN.P$10, PT_123_IN.P$12, PT_123_IN.P$2, PT_123_IN.P$4, PT_123_IN.P$6, PT_123_IN.P$8, TC_PT4_IN.P$12, TC_PT4_IN.P$6
- net +3V3_LC: now also LC_EN/CAL.1; no longer CAL1.1
- net ADC1_A0: now also C31.2, IC5.6, RF1.1
- net ADC1_A1: now also C13.2, IC10.6, RF2.1
- net ADC1_A2: now also C33.2, IC11.6, RF3.1
- net ADC1_A3: now also C35.2, IC12.6, RF4.1
- net ADC2_A4: now also THERMOCOUPLES.A1, THERMOCOUPLES.B1; no longer TC_PT4_IN.P$10, TC_PT4_IN.P$4
- net ADC2_A5: now also THERMOCOUPLES.A2, THERMOCOUPLES.B2; no longer TC_PT4_IN.P$3, TC_PT4_IN.P$9
- net ADC2_A6: now also THERMOCOUPLES.A3, THERMOCOUPLES.B3; no longer TC_PT4_IN.P$2, TC_PT4_IN.P$8
- net ADC2_A7: now also THERMOCOUPLES.A4, THERMOCOUPLES.B4; no longer TC_PT4_IN.P$1, TC_PT4_IN.P$7
- net CAL: now also IC5.8, LC_EN/CAL.2, RPD1.1
- net CTRL_SOLENOID_4: now also RPI_GPIO.18
- net LC_1_OUT+: now also LC1/2.A3, LC1/2.B3; no longer U$4.A3, U$4.B3
- net LC_1_OUT-: now also LC1/2.A4, LC1/2.B4; no longer U$4.A4, U$4.B4
- net LC_2_OUT+: now also LC1/2.A1, LC1/2.B1; no longer U$4.A1, U$4.B1
- net LC_2_OUT-: now also LC1/2.A2, LC1/2.B2; no longer U$4.A2, U$4.B2
- net LC_3_OUT+: now also LC3/4.A3, LC3/4.B3; no longer U$1.A3, U$1.B3
- net LC_3_OUT-: now also LC3/4.A4, LC3/4.B4; no longer U$1.A4, U$1.B4
- net LC_4_OUT+: now also LC3/4.A1, LC3/4.B1; no longer U$1.A1, U$1.B1
- net LC_4_OUT-: now also LC3/4.A2, LC3/4.B2; no longer U$1.A2, U$1.B2
- net PT1_VS-: now also PT1/2.A2, PT1/2.B2; no longer PT_123_IN.P$11, PT_123_IN.P$5
- net PT2_VS-: now also PT1/2.A4, PT1/2.B4; no longer PT_123_IN.P$3, PT_123_IN.P$9
- net PT3_VS-: now also PT3/4.A2, PT3/4.B2; no longer PT_123_IN.P$1, PT_123_IN.P$7
- net PT4_VS-: now also PT3/4.A4, PT3/4.B4; no longer TC_PT4_IN.P$11, TC_PT4_IN.P$5
Routing:
- net GND: track 0.00 -> 28.0 mm, vias 0 -> 5
- net +12V: track 153.5 -> 132.3 mm, vias 0 -> 1
- net SOLENOID_1_NEGATIVE: track 49.0 -> 65.5 mm
- net RELAY_NEGATIVE: track 36.2 -> 52.3 mm
- net SOLENOID_2_NEGATIVE: track 71.9 -> 85.7 mm
- net SOLENOID_3_NEGATIVE: track 88.2 -> 101.9 mm
- net +10V: track 63.1 -> 52.6 mm, vias 0 -> 1
- net N$15: track 8.20 -> 0.00 mm
- net +5V: track 54.8 -> 60.1 mm
- net SOLENOID_4_NEGATIVE: track 24.9 -> 20.0 mm
- net +3V3: track 51.6 -> 47.7 mm
- net +12V_DEBUG: track 28.4 -> 29.9 mm
